Commit message: rotation correction

File: xacro/main.urdf.xacro (robot description, xacro)
@@ -36,5 +36,5 @@
 		<parent link="origin_link" />
 		<child link="base_link" />
-		<origin xyz="0 0 0.0175" />
+		<origin xyz="0 0 0.0175" rpy="0 0 ${-pi/2}"/>
 	</joint>
 	<xacro:layer1

Commit message: navigation in development

File: xacro/main.urdf.xacro (robot description, xacro)
@@ -8,4 +8,5 @@
 	<xacro:property name="base_r" value="${0.063}" />
 	<link name="origin_link"/>
+	<link name="map"/>
 	<link name="base_link">
 		<inertial>
@@ -37,4 +38,11 @@
 		<child link="base_link" />
 		<origin xyz="0 0 0.0175" rpy="0 0 ${-pi/2}"/>
+	</joint>
+	<joint
+		name="map_joint"
+		type="fixed">
+		<parent link="origin_link" />
+		<child link="map" />
+		<origin xyz="0 0 0" rpy="0 0 0"/>
 	</joint>
 	<xacro:layer1
@@ -71,3 +79,55 @@
 		</plugin>
 	</gazebo>
+	<!-- Laser Scan -->
+	<link name="hokuyo_link">
+		<collision>
+			<origin xyz="0 0 0" rpy="0 0 0"/>
+			<geometry>
+				<box size="0.1 0.1 0.1"/>
+			</geometry>
+		</collision>
+		<visual>
+			<origin xyz="0 0 0" rpy="0 0 0"/>
+			<geometry>
+				<box size="0.1 0.1 0.1"/>
+			</geometry>
+		</visual>
+		<inertial>
+			<mass value="1e-5" />
+			<origin xyz="0 0 0" rpy="0 0 0"/>
+			<inertia ixx="1e-6" ixy="0" ixz="0" iyy="1e-6" iyz="0" izz="1e-6" />
+		</inertial>
+	</link>
+	<joint name="hokuyo_joint" type="fixed">
+		<axis xyz="0 1 0" />
+		<origin xyz="0 0 0.2" rpy="0 0 0"/>
+		<parent link="origin_link"/>
+		<child link="hokuyo_link"/>
+	</joint>
+	<gazebo reference="hokuyo_link">
+		<sensor type="gpu_ray" name="hokuyo">
+			<pose>0 0 0 0 0 0</pose>
+			<visualize>false</visualize>
+			<update_rate>40</update_rate>
+			<ray>
+				<scan>
+					<horizontal>
+						<samples>720</samples>
+						<resolution>1</resolution>
+						<min_angle>-1.570796</min_angle>
+						<max_angle>1.570796</max_angle>
+					</horizontal>
+				</scan>
+				<range>
+					<min>0.10</min>
+					<max>30.0</max>
+					<resolution>0.01</resolution>
+				</range>
+			</ray>
+			<plugin name="gpu_laser" filename="libgazebo_ros_gpu_laser.so">
+				<topicName>/scan</topicName>
+				<frameName>hokuyo_link</frameName>
+			</plugin>
+		</sensor>
+	</gazebo>
 </robot>

Commit message: scanner poorly working

File: xacro/main.urdf.xacro (robot description, xacro)
@@ -80,5 +80,5 @@
 	</gazebo>
 	<!-- Laser Scan -->
-	<link name="hokuyo_link">
+	<link name="/robot_1/hokuyo_link">
 		<collision>
 			<origin xyz="0 0 0" rpy="0 0 0"/>
@@ -102,9 +102,9 @@
 		<axis xyz="0 1 0" />
 		<origin xyz="0 0 0.2" rpy="0 0 0"/>
-		<parent link="origin_link"/>
-		<child link="hokuyo_link"/>
+		<parent link="base_link"/>
+		<child link="/robot_1/hokuyo_link"/>
 	</joint>
-	<gazebo reference="hokuyo_link">
-		<sensor type="gpu_ray" name="hokuyo">
+	<gazebo reference="/robot_1/hokuyo_link">
+		<sensor type="ray" name="hokuyo">
 			<pose>0 0 0 0 0 0</pose>
 			<visualize>false</visualize>
@@ -125,7 +125,8 @@
 				</range>
 			</ray>
-			<plugin name="gpu_laser" filename="libgazebo_ros_gpu_laser.so">
+			<plugin name="gazebo_ros_laser" filename="libgazebo_ros_laser.so">
 				<topicName>/scan</topicName>
 				<frameName>hokuyo_link</frameName>
+           	 		<robotNamespace>robot_1</robotNamespace>
 			</plugin>
 		</sensor>

Commit message: loading map and laser sensor, map and odom frames have strange behaviour

File: xacro/main.urdf.xacro (robot description, xacro)
@@ -8,5 +8,5 @@
 	<xacro:property name="base_r" value="${0.063}" />
 	<link name="origin_link"/>
-	<link name="map"/>
+	<!--link name="map"/-->
 	<link name="base_link">
 		<inertial>
@@ -39,5 +39,5 @@
 		<origin xyz="0 0 0.0175" rpy="0 0 ${-pi/2}"/>
 	</joint>
-	<joint
+	<!--joint
 		name="map_joint"
 		type="fixed">
@@ -45,5 +45,5 @@
 		<child link="map" />
 		<origin xyz="0 0 0" rpy="0 0 0"/>
-	</joint>
+	</joint-->
 	<xacro:layer1
 		height="0.025"/>
@@ -80,5 +80,5 @@
 	</gazebo>
 	<!-- Laser Scan -->
-	<link name="/robot_1/hokuyo_link">
+	<link name="hokuyo_link">
 		<collision>
 			<origin xyz="0 0 0" rpy="0 0 0"/>
@@ -103,7 +103,7 @@
 		<origin xyz="0 0 0.2" rpy="0 0 0"/>
 		<parent link="base_link"/>
-		<child link="/robot_1/hokuyo_link"/>
+		<child link="hokuyo_link"/>
 	</joint>
-	<gazebo reference="/robot_1/hokuyo_link">
+	<gazebo reference="hokuyo_link">
 		<sensor type="ray" name="hokuyo">
 			<pose>0 0 0 0 0 0</pose>
@@ -126,6 +126,6 @@
 			</ray>
 			<plugin name="gazebo_ros_laser" filename="libgazebo_ros_laser.so">
-				<topicName>front/scan</topicName>
-				<frameName>hokuyo_link</frameName>
+				<topicName>scan</topicName>
+				<frameName>/hokuyo_link</frameName>
            	 		<robotNamespace>robot_1</robotNamespace>
 			</plugin>

Commit message: global trajectory working

File: xacro/main.urdf.xacro (robot description, xacro)
@@ -80,5 +80,5 @@
 	</gazebo>
 	<!-- Laser Scan -->
-	<link name="hokuyo_link">
+	<!--link name="hokuyo_link">
 		<collision>
 			<origin xyz="0 0 0" rpy="0 0 0"/>
@@ -131,4 +131,4 @@
 			</plugin>
 		</sensor>
-	</gazebo>
+	</gazebo-->
 </robot>
